File: lumberjack-pro-keyboard.kicad_pcb (KiCad board)
At the start: 2 copper layers, 284.7 x 94.2 mm, 149 parts, among them J1 USB, J3 JST, J4 JST, SW1 RESET, U1 Frood/nice!nano

Commit message: Update silkscreen
Parts:
- LOGO2: value Lumberjack Pro Frood -> Lumberjack Pro
- MX5: value SW_Push+EC11 -> SW_Push
Other:
- board text added: "DANGER! DO NOT USE WITH BATTERY!"
- board text added: "rev1.0.5 01/2026"
- board text removed: "JLCJLCJLCJLC"
- board text removed: "rev1.0 06/2024"
